File: SENSOR_PERIPHERIAL.brd (EAGLE design)
At the start: 160 x 100 mm, 0 parts

Commit message: added some initial frameworks
Parts:
- added JP1: (no value), SparkFun-Connectors:1X03_SMD_RA_MALE
- added U$1: BMP085, SparkFun-Sensors:BMP085
- added U$2: SHT1XSMD, SparkFun-Sensors:SHT1X
- added U1: VENUS638FLPX-L, SparkFun-RF:VENUS638FLPX
Connections:
- new net 5V: JP1.1
- new net GND: JP1.3, U$1.1, U$2.1
- new net ONE_WIRE_TEMP: JP1.2
- new net VDD: U$2.4
- new net VDDA: U$1.3
- new net VDDD: U$1.4
Changed lines of the file:
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@@
 <?xml version="1.0" encoding="utf-8"?>
 <!DOCTYPE eagle SYSTEM "eagle.dtd">
-<eagle version="6.1">
+<eagle version="6.4">
 <drawing>
 <settings>
@@
 <layer number="106" name="bPlate" color="7" fill="1" visible="no" active="yes"/>
 <layer number="107" name="Crop" color="7" fill="1" visible="no" active="yes"/>
+<layer number="108" name="tplace-old" color="10" fill="1" visible="yes" active="yes"/>
+<layer number="109" name="ref-old" color="11" fill="1" visible="yes" active="yes"/>
 <layer number="116" name="Patch_BOT" color="9" fill="4" visible="no" active="yes"/>
 <layer number="121" name="_tsilk" color="7" fill="1" visible="no" active="yes"/>
@@
 <layer number="144" name="Drill_legend" color="7" fill="1" visible="no" active="yes"/>
 <layer number="151" name="HeatSink" color="7" fill="1" visible="no" active="yes"/>
+<layer number="199" name="Contour" color="7" fill="1" visible="yes" active="yes"/>
 <layer number="200" name="200bmp" color="1" fill="10" visible="no" active="yes"/>
 <layer number="201" name="201bmp" color="2" fill="10" visible="no" active="yes"/>
@@
 </class>
 </classes>
-<designrules>
+<designrules name="default">
 <description language="de">&lt;b&gt;EAGLE Design Rules&lt;/b&gt;
 &lt;p&gt;
@@
 </autorouter>
 <elements>
+<element name="U1" library="SparkFun-RF" package="VENUS638FLPX" value="VENUS638FLPX-L" x="6.35" y="-6.35"/>
+<element name="JP1" library="SparkFun-Connectors" package="1X03_SMD_RA_MALE" value="" x="-5.08" y="-3.81">
+<attribute name="PROD_ID" value="CONN-10925" x="-5.08" y="-3.81" size="1.778" layer="27" display="off"/>
+</element>
+<element name="U$1" library="SparkFun-Sensors" package="BMP085" value="BMP085" x="-5.08" y="-15.24"/>
+<element name="U$2" library="SparkFun-Sensors" package="SHT1X" value="SHT1XSMD" x="-12.7" y="-13.97"/>
 </elements>
 <signals>
+<signal name="ONE_WIRE_TEMP">
+<contactref element="JP1" pad="2"/>
+</signal>
+<signal name="5V">
+<contactref element="JP1" pad="1"/>
+</signal>
+<signal name="GND">
+<contactref element="JP1" pad="3"/>
+<contactref element="U$1" pad="1"/>
+<contactref element="U$2" pad="1"/>
+<wire x1="-7.145" y1="-13.97" x2="-15.367" y2="-12.065" width="0" layer="19" extent="1-1"/>
+<wire x1="-2.54" y1="1.19" x2="-7.145" y2="-13.97" width="0" layer="19" extent="1-1"/>
+</signal>
+<signal name="VDDD">
+<contactref element="U$1" pad="4"/>
+</signal>
+<signal name="VDDA">
+<contactref element="U$1" pad="3"/>
+</signal>
+<signal name="VDD">
+<contactref element="U$2" pad="4"/>
+</signal>
 </signals>
 </board>
